Commit message: removed unnecessary things

File: gazebo/gazebo.urdf.xacro (robot description, xacro)
@@ -1,50 +1,24 @@
-<?xml version="1.0"?>
-<!--
-  Copyright (c) 2011, PAL Robotics, S.L.
-  All rights reserved.
-  This work is licensed under the Creative Commons Attribution-NonCommercial-NoDerivs 3.0 Unported License.
-  To view a copy of this license, visit http://creativecommons.org/licenses/by-nc-nd/3.0/ or send a letter to
-  Creative Commons, 444 Castro Street, Suite 900, Mountain View, California, 94041, USA.
--->
-<robot name="lobot">
+<?xml version="1.0" ?>
+<robot xmlns:xacro="http://ros.org/wiki/xacro" name="lobot">
   <gazebo>
-    <plugin filename="libgazebo_ros_control.so" name="gazebo_ros_control">
-      <robotNamespace>/lobot</robotNamespace>
-      <robotSimType>gazebo_ros_control/DefaultRobotHWSim</robotSimType>
-    </plugin>
-    <plugin filename="libgazebo_ros_p3d.so" name="gazebo_ros_p3d">
-      <bodyName>base_link</bodyName>
-      <topicName>ground_truth_odom</topicName>
-      <alwaysOn>true</alwaysOn>
-      <updateRate>100.0</updateRate>
+    <plugin filename="libmy_joint_state_publisher.so" name="my_joint_state_publisher">
+      <robot_name>lobot</robot_name>
+      <update_rate>100</update_rate>
     </plugin>
   </gazebo>
   <gazebo>
-    <plugin filename="libgazebo_ros_force.so" name="gazebo_ros_force">
-      <bodyName>base_link</bodyName>
-      <topicName>base_link_wrench</topicName>
+    <plugin filename="librobot_plugin.so" name="robot_plugin_lobot">
+      <robot_name>lobot</robot_name>
+      <update_rate>100</update_rate>
     </plugin>
   </gazebo>
-  <gazebo>
-    <plugin filename="libgazebo_world_odometry.so" name="gazebo_ros_odometry">
-      <frameName>base_link</frameName>
-      <topicName>floating_base_pose_simulated</topicName>
-    </plugin>
-  </gazebo>
-  <gazebo reference="r_foot">
-    <mu1>0.9</mu1>
-    <mu2>0.9</mu2>
-    <fdir1>1 0 0</fdir1>
-    <maxVel>1.0</maxVel>
-    <minDepth>0.003</minDepth>
-  </gazebo>
-  <gazebo reference="l_foot">
-    <mu1>0.9</mu1>
-    <mu2>0.9</mu2>
-    <fdir1>1 0 0</fdir1>
-    <maxVel>1.0</maxVel>
-    <minDepth>0.003</minDepth>
+  <gazebo reference="IMU_link">
+    <sensor type="imu" name="IMU_lobot">
+      <always_on>true</always_on>
+      <update_rate>10.0</update_rate>
+      <plugin filename="libgazebo_ros_imu_sensor.so" name="lobot_IMU_controller"></plugin>
+    </sensor>
   </gazebo>
   <!-- define global properties -->
-  <property name="M_PI" value="3.1415926535897931" />
+  <xacro:property name="M_PI" value="3.1415926535897931" />
 </robot>

File: urdf/arm/arm.transmission.xacro (robot description, xacro)
@@ -1,5 +1,5 @@
 <?xml version="1.0"?>
 <robot name="lobot" xmlns:xacro="http://ros.org/wiki/xacro">
-  <xacro:macro name="lobot_leg_transmission" params="name side number reduction" >
+  <xacro:macro name="lobot_arm_transmission" params="name side number reduction" >
     <transmission name="${name}_${side}_${number}_trans">
       <type>transmission_interface/SimpleTransmission</type>
@@ -8,5 +8,6 @@
       </actuator>
       <joint name="${name}_${side}_${number}_joint">
-        <hardwareInterface>hardware_interface/JointCommandHandle</hardwareInterface>
+        <!-- <hardwareInterface>hardware_interface/PositionJointInterface</hardwareInterface> -->
+        <hardwareInterface>hardware_interface/EffortJointInterface</hardwareInterface>
       </joint>
     </transmission>

File: urdf/leg/leg.urdf.xacro (robot description, xacro)
@@ -1,12 +1,9 @@
-<?xml version="1.0"?>
+<?xml version="1.0" ?>
 <!--
-  Copyright (c) 2011-2012, PAL Robotics, S.L.
+  Author: Poh Zhi-Ee (zhiee.poh@httechnology.com)
+  Copyright (c) 2019, SIW Manufacturing Sdn. Bhd.
   All rights reserved.
-  This work is licensed under the Creative Commons Attribution-NonCommercial-NoDerivs 3.0 Unported License.
-  To view a copy of this license, visit http://creativecommons.org/licenses/by-nc-nd/3.0/ or send a letter to
-  Creative Commons, 444 Castro Street, Suite 900, Mountain View, California, 94041, USA.
 -->
-<robot name="lobot"
-    xmlns:xacro="http://ros.org/wiki/xacro">
+<robot name="lobot" xmlns:xacro="http://ros.org/wiki/xacro">
     <!--File includes-->
     <xacro:include filename="$(find lobot_description)/urdf/leg/leg.transmission.xacro" />
@@ -33,32 +30,168 @@
         <link name="leg_${side}_1_link">
             <inertial>
-                <mass value="1.02901"/>
-                <origin xyz="-0.02571 0 0.02557" rpy="0 0 0"/>
-                <inertia ixx="0.00132187534" ixy="0.00000001514" ixz="0.00040022268" iyy="0.0018528617" iyz="0.00000050713" izz="0.00084231334"/>
-            </inertial>
-            <visual>
-                <origin rpy="0 0 0" xyz="0 0 0"/>
-                <geometry>
-                    <box size="0.15 0.10 0.20"/>
-                </geometry>
-                <material name="LightGrey" />
-            </visual>
-            <collision>
-                <origin xyz="0 0 0" rpy="0 0 0" />
-                <geometry>
-                    <box size="0.15 0.10 0.20"/>
-                    <!-- <box size="0.3 0.35 0.14"/> -->
+                <mass value="0.02901" />
+                <origin xyz="0 0 0" rpy="0.0 0.0 0.0" />
+                <inertia ixx="0.00132187534" ixy="0.00000001514" ixz="0.00040022268" iyy="0.0018528617" iyz="0.00000050713" izz="0.00084231334" />
+            </inertial>
+            <visual>
+                <origin rpy="0 ${90*deg_to_rad} 0" xyz="0 0 0" />
+                <geometry>
+                    <cylinder radius="0.01" length="0.02" />
+                </geometry>
+                <material name="LightGrey" />
+            </visual>
+            <collision>
+                <origin rpy="0 ${90*deg_to_rad} 0" xyz="0 0 0" />
+                <geometry>
+                    <cylinder radius="0.01" length="0.02" />
                 </geometry>
             </collision>
         </link>
         <joint name="leg_${side}_1_joint" type="revolute">
-            <origin xyz="0  ${-reflect*0.075} -0.14353" rpy="0 0 0"/>
-            <axis xyz="0 0 1"/>
-            <parent link="${parent}"/>
-            <child link="leg_${side}_1_link"/>
+            <origin xyz="0  ${-reflect*0.0315} -0.0475" rpy="0 0 0" />
+            <axis xyz="1 0 0" />
+            <parent link="${parent}" />
+            <child link="leg_${side}_1_link" />
             <limit lower="-1.57" upper="1.57" effort="50" velocity="4" />
-            <dynamics friction="${leg_friction}" damping="${leg_damping}"/>
-            <!-- <limit lower="${-37.5*deg_to_rad + reflect*7.5*deg_to_rad}" upper="${37.5*deg_to_rad + reflect*7.5*deg_to_rad}" effort="${leg_1_joint_effort}" velocity="${leg_1_joint_max_vel}" /> -->
-            <!-- <safety_controller k_position="100" k_velocity="100" soft_lower_limit="${-75*deg_to_rad + reflect*7.5*deg_to_rad + leg_eps}" soft_upper_limit="${ 37.5*deg_to_rad + reflect*7.5*deg_to_rad - leg_eps}" /> -->
+        </joint>
+        <link name="leg_${side}_2_link">
+            <inertial>
+                <mass value="0.069621" />
+                <origin xyz="0 0 0" rpy="0.0 0.0 0.0" />
+                <inertia ixx="0.0008416476" ixy="-0.00000268743" ixz="0.00000667199" iyy="0.00039794844" iyz="0.00002668971" izz="0.00084196694" />
+            </inertial>
+            <visual>
+                    <origin rpy="0 ${26.565*deg_to_rad} 0" xyz="0.02 0 0" />
+                <geometry>
+                    <!-- <cylinder radius="0.01" length="0.02" /> -->
+                    <box size="0.02 0.04 0.02" />
+                </geometry>
+                <material name="LightGrey" />
+            </visual>
+            <collision>
+                <origin rpy="0 ${26.565*deg_to_rad} 0" xyz="0.02 0 0" />
+                <geometry>
+                    <!-- <cylinder radius="0.01" length="0.02" /> -->
+                    <box size="0.03 0.03 0.02" />
+                </geometry>
+            </collision>
+        </link>
+        <joint name="leg_${side}_2_joint" type="revolute">
+            <origin xyz="0 0 -0.04707" rpy="0 0 0" />
+            <axis xyz="0 1 0" />
+            <parent link="leg_${side}_1_link" />
+            <child link="leg_${side}_2_link" />
+            <limit lower="${-22.5*deg_to_rad - reflect*7.5*deg_to_rad}" upper="${22.5*deg_to_rad - reflect*7.5*deg_to_rad}" effort="${leg_2_joint_effort}" velocity="${leg_2_joint_max_vel}" />
+        </joint>
+        <link name="leg_${side}_3a_link">
+            <inertial>
+                <mass value="0.04" />
+                <origin xyz="0 0 0" rpy="0.0 0.0 0.0" />
+                <inertia ixx="0.0008416476" ixy="-0.00000268743" ixz="0.00000667199" iyy="0.00039794844" iyz="0.00002668971" izz="0.00084196694" />
+            </inertial>
+            <visual>
+                <origin rpy="0 0 0" xyz="0 0 0.004" />
+                <geometry>
+                    <box size="0.02 0.04 0.025" />
+                </geometry>
+                <material name="LightGrey" />
+            </visual>
+            <collision>
+                <origin rpy="0 0 0" xyz="0 0 0.004" />
+                <geometry>
+                    <box size="0.02 0.04 0.025" />
+                </geometry>
+            </collision>
+        </link>
+        <joint name="leg_${side}_3a_joint" type="fixed">
+            <origin xyz="0.04104 0 -0.020" rpy="0 0 0" />
+            <parent link="leg_${side}_2_link" />
+            <child link="leg_${side}_3a_link" />
+        </joint>
+        <link name="leg_${side}_3_link">
+            <inertial>
+                <mass value="0.05" />
+                <origin xyz="0 0 0" rpy="0.0 0.0 0.0" />
+                <inertia ixx="0.0008416476" ixy="-0.00000268743" ixz="0.00000667199" iyy="0.00039794844" iyz="0.00002668971" izz="0.00084196694" />
+            </inertial>
+            <visual>
+                <origin rpy="0 0 0" xyz="0 0 -0.02" />
+                <geometry>
+                    <box size="0.02 0.04 0.04" />
+                </geometry>
+                <material name="LightGrey" />
+            </visual>
+            <collision>
+                <origin rpy="0 0 0" xyz="0 0 -0.02" />
+                <geometry>
+                    <box size="0.02 0.04 0.04" />
+                </geometry>
+            </collision>
+        </link>
+        <joint name="leg_${side}_3_joint" type="revolute">
+            <origin xyz="0 0 -0.02477" rpy="0 0 0" />
+            <axis xyz="0 1 0" />
+            <parent link="leg_${side}_3a_link" />
+            <child link="leg_${side}_3_link" />
+            <!-- <dynamics friction="${leg_friction}" damping="${leg_damping}" /> -->
+            <limit lower="${ -100.0 * deg_to_rad}" upper="${45 * deg_to_rad}" effort="${leg_3_joint_effort}" velocity="${leg_3_joint_max_vel}" />
+            <!-- <safety_controller k_position="100" k_velocity="100" soft_lower_limit="${-100.0 * deg_to_rad + leg_eps}" soft_upper_limit="${  45.0 * deg_to_rad - leg_eps}" /> -->
+        </joint>
+        <link name="leg_${side}_4_link">
+            <inertial>
+                <mass value="0.06" />
+                <origin xyz="0 0 0" rpy="0.0 0.0 0.0" />
+                <inertia ixx="0.0008416476" ixy="-0.00000268743" ixz="0.00000667199" iyy="0.00039794844" iyz="0.00002668971" izz="0.00084196694" />
+            </inertial>
+            <visual>
+                <origin rpy="${90*deg_to_rad} 0 0" xyz="0 0 0" />
+                <geometry>
+                    <cylinder radius="0.01" length="0.02" />
+                </geometry>
+                <material name="LightGrey" />
+            </visual>
+            <collision>
+                <origin rpy="${90*deg_to_rad} 0 0" xyz="0 0 0" />
+                <geometry>
+                    <cylinder radius="0.01" length="0.02" />
+                </geometry>
+            </collision>
+        </link>
+        <joint name="leg_${side}_4_joint" type="revolute">
+            <origin xyz="0 0 -0.05856" rpy="0 0 0" />
+            <axis xyz="0 1 0" />
+            <parent link="leg_${side}_3_link" />
+            <child link="leg_${side}_4_link" />
+            <dynamics friction="${leg_friction}" damping="${leg_damping}" />
+            <limit lower="${ -100.0 * deg_to_rad}" upper="${45 * deg_to_rad}" effort="${leg_3_joint_effort}" velocity="${leg_3_joint_max_vel}" />
+            <safety_controller k_position="100" k_velocity="100" soft_lower_limit="${-100.0 * deg_to_rad + leg_eps}" soft_upper_limit="${  45.0 * deg_to_rad - leg_eps}" />
+        </joint>
+        <link name="leg_${side}_5_link">
+            <inertial>
+                <mass value="0.05" />
+                <origin xyz="0 0 0" rpy="0.0 0.0 0.0" />
+                <inertia ixx="0.0008416476" ixy="-0.00000268743" ixz="0.00000667199" iyy="0.00039794844" iyz="0.00002668971" izz="0.00084196694" />
+            </inertial>
+            <visual>
+                <origin rpy="0 0 0" xyz="0 0 -0.005" />
+                <geometry>
+                    <!-- <cylinder radius="0.01" length="0.02" /> -->
+                    <box size="0.095 0.07 0.01" />
+                </geometry>
+                <material name="LightGrey" />
+            </visual>
+            <collision>
+                <origin rpy="0 0 0" xyz="0 0 -0.005" />
+                <geometry>
+                    <box size="0.095 0.07 0.01" />
+                </geometry>
+            </collision>
+        </link>
+        <joint name="leg_${side}_5_joint" type="revolute">
+            <origin xyz="0 0 -0.04707" rpy="0 0 0" />
+            <axis xyz="1 0 0" />
+            <parent link="leg_${side}_4_link" />
+            <child link="leg_${side}_5_link" />
+            <limit lower="${ -100.0 * deg_to_rad}" upper="${45 * deg_to_rad}" effort="${leg_3_joint_effort}" velocity="${leg_3_joint_max_vel}" />
         </joint>
         <gazebo reference="leg_${side}_1_link">
@@ -66,21 +199,8 @@
             <mu2>0.9</mu2>
         </gazebo>
-        <!-- contact model for foot surface -->
-        <!-- <gazebo reference="leg_${side}_6_link">
-            <kp>1000000.0</kp>
-            <kd>100.0</kd>
-            <mu1>1.0</mu1>
-            <mu2>1.0</mu2>
-            <fdir1>0 0 1</fdir1>
-            <maxVel>1.0</maxVel>
-            <minDepth>0.00</minDepth>
-            <implicitSpringDamper>1</implicitSpringDamper>
-        </gazebo> -->
-        <!--force torque sensor -->
-        <!--xacro:reemc_force_torque_sensor name="leg_${side}_6_link" update_rate="100.0"/-->
         <gazebo reference="leg_${side}_1_joint">
             <implicitSpringDamper>1</implicitSpringDamper>
         </gazebo>
-        <!-- <gazebo reference="leg_${side}_2_joint">
+        <gazebo reference="leg_${side}_2_joint">
             <implicitSpringDamper>1</implicitSpringDamper>
         </gazebo>
@@ -91,4 +211,5 @@
             <implicitSpringDamper>1</implicitSpringDamper>
         </gazebo>
+        <!--
         <gazebo reference="leg_${side}_5_joint">
             <implicitSpringDamper>1</implicitSpringDamper>
@@ -99,9 +220,11 @@
         </gazebo> -->
         <xacro:lobot_leg_transmission name="${name}" side="${side}" number="1" reduction="${leg_reduction}" />
-        <!-- <xacro:reemc_leg_simple_transmission name="${name}" side="${side}" number="2" reduction="${leg_reduction}" />
-        <xacro:reemc_leg_simple_transmission name="${name}" side="${side}" number="3" reduction="${leg_reduction}" />
-        <xacro:reemc_leg_simple_transmission name="${name}" side="${side}" number="4" reduction="${leg_reduction}" />
-        <xacro:reemc_leg_simple_transmission name="${name}" side="${side}" number="5" reduction="${leg_reduction}" />
-        <xacro:reemc_leg_simple_transmission name="${name}" side="${side}" number="6" reduction="${leg_reduction}" /> -->
+        <xacro:lobot_leg_transmission name="${name}" side="${side}" number="2" reduction="${leg_reduction}" />
+        <xacro:lobot_leg_transmission name="${name}" side="${side}" number="3" reduction="${leg_reduction}" />
+        <xacro:lobot_leg_transmission name="${name}" side="${side}" number="4" reduction="${leg_reduction}" />
+        <!--
+        <xacro:lobot_leg_simple_transmission name="${name}" side="${side}" number="5" reduction="${leg_reduction}" />
+        <xacro:lobot_leg_simple_transmission name="${name}" side="${side}" number="6" reduction="${leg_reduction}" />
+        -->
     </xacro:macro>
 </robot>
