Commit message: updated joint limits

File: robots/biped.urdf (robot description, URDF)
Before this commit: robot lobot, 23 links, 22 joints
Links:
- link leg_left_2_link: geometry collision box size=0.02 0.04 0.02; visual box size=0.02 0.04 0.02
- link leg_right_2_link: geometry collision box size=0.02 0.04 0.02; visual box size=0.02 0.04 0.02
Joints:
- joint leg_left_1_joint: limit lower=-1.57 upper=1.57 effort=50 velocity=4 -> lower=-1.2 upper=1.2 effort=50 velocity=4
- joint leg_left_2_joint: limit lower=-0.261799387799 upper=0.523598775598 effort=64.0 velocity=2.27 -> lower=-1.2 upper=1.2 effort=50 velocity=4
- joint leg_left_3_joint: limit lower=-1.74532925199 upper=0.785398163397 effort=55.7 velocity=3.64 -> lower=-1.2 upper=1.2 effort=50 velocity=4
- joint leg_left_4_joint: limit lower=-1.74532925199 upper=0.785398163397 effort=55.7 velocity=3.64 -> lower=-1.2 upper=1.2 effort=50 velocity=4
- joint leg_left_5_joint: limit lower=-1.74532925199 upper=0.785398163397 effort=55.7 velocity=3.64 -> lower=-1.2 upper=1.2 effort=50 velocity=4
- joint leg_right_1_joint: limit lower=-1.57 upper=1.57 effort=50 velocity=4 -> lower=-1.2 upper=1.2 effort=50 velocity=4
- joint leg_right_2_joint: limit lower=-0.523598775598 upper=0.261799387799 effort=64.0 velocity=2.27 -> lower=-1.2 upper=1.2 effort=50 velocity=4
- joint leg_right_3_joint: limit lower=-1.74532925199 upper=0.785398163397 effort=55.7 velocity=3.64 -> lower=-1.2 upper=1.2 effort=50 velocity=4
- joint leg_right_4_joint: limit lower=-1.74532925199 upper=0.785398163397 effort=55.7 velocity=3.64 -> lower=-1.2 upper=1.2 effort=50 velocity=4
- joint leg_right_5_joint: limit lower=-1.74532925199 upper=0.785398163397 effort=55.7 velocity=3.64 -> lower=-1.2 upper=1.2 effort=50 velocity=4
