Commit message: update mass properties

File: robots/arm_standalone.urdf (robot description, URDF)
Before this commit: robot lobot, 8 links, 7 joints
Links:
- removed link arm_2_interm_link
- added link arm_bracket_1, mass 0.00658; visual box size=0.052 0.025 0.002
- added link arm_bracket_2, mass 0.01175; collision box size=0.055 0.002 0.025; visual box size=0.055 0.002 0.025
- link arm_2_link: mass 0.06 -> 0.0618
- link arm_3_link: mass 0.06 -> 0.0618
- link grip_link_1: mass 0.005 -> 0.01023; geometry collision box size=0.04 0.055 0.001; visual box size=0.04 0.055 0.001
- link grip_link_2: geometry collision box size=0.04 0.017 0.001; visual box size=0.04 0.017 0.001
- link grip_link_3: geometry collision box size=0.04 0.001 0.007; visual box size=0.04 0.001 0.007
Joints:
- added joint arm_bracket_2_joint: type fixed, parent arm_2_link, child arm_bracket_2, origin xyz=0 -0.03653 0 rpy=0 0 0
- joint arm_1_joint: child arm_2_interm_link -> arm_bracket_1; origin xyz=0 0.01 0.052 rpy=0 0 0 -> xyz=0 0.01 0.0 rpy=0 0 0
- joint arm_2_joint: origin xyz=0 0 0 rpy=0 0 0 -> xyz=0 0 0.052 rpy=0 0 0; parent arm_2_interm_link -> arm_bracket_1

Commit message: add gazebo plugins

File: robots/arm_standalone.urdf (robot description, URDF)
Before this commit: robot lobot, 9 links, 8 joints
Links:
- link arm_bracket_1: geometry collision box size=0.052 0.025 0.002; visual box size=0.052 0.025 0.002

Commit message: update joint limits

File: robots/arm_standalone.urdf (robot description, URDF)
Before this commit: robot lobot, 9 links, 8 joints
Joints:
- joint arm_1_joint: limit lower=-2.356 upper=2.356 effort=50 velocity=40 -> lower=-2.356 upper=2.356 effort=20 velocity=10
- joint arm_2_joint: limit lower=-2.356 upper=2.356 effort=50 velocity=40 -> lower=-1.570796 upper=1.570796 effort=20 velocity=20
- joint arm_3_joint: limit lower=-2.356 upper=2.356 effort=50 velocity=40 -> lower=-1.570796 upper=1.570796 effort=10 velocity=10

Commit message: Update plugin names, add contact plugin and effort limits
librobot_plugin.so -> librobot_control_p;lugin.so

arm_standalone effort limits now allows for proper terminal velocity such that control is good

File: robots/arm_standalone.urdf (robot description, URDF)
Before this commit: robot lobot, 9 links, 8 joints
Joints:
- joint arm_1_joint: limit lower=-2.356 upper=2.356 effort=20 velocity=10 -> lower=-2.356 upper=2.356 effort=3.5 velocity=10
- joint arm_2_joint: limit lower=-1.570796 upper=1.570796 effort=20 velocity=20 -> lower=-1.570796 upper=1.570796 effort=3 velocity=20
- joint arm_3_joint: limit lower=-1.570796 upper=1.570796 effort=10 velocity=10 -> lower=-1.570796 upper=1.570796 effort=3 velocity=10

Commit message: Update to add visual only point to indicate arm gripper end
 Also removes simulation rate limiter in gym training world

File: robots/arm_standalone.urdf (robot description, URDF)
Before this commit: robot lobot, 9 links, 8 joints
Links:
- added link grip_end_point, mass 0.0000001; visual sphere radius=0.001
Joints:
- added joint grip_joint_4: type fixed, parent grip_link_3, child grip_end_point, origin xyz=0 -0.0005 -0.0035 rpy=0 0 0

Commit message: Update joint2 limits
Changed maximum to 0.5 radians because any more will cause collision with itself

File: robots/arm_standalone.urdf (robot description, URDF)
Before this commit: robot lobot, 10 links, 9 joints
Joints:
- joint arm_2_joint: limit lower=-1.570796 upper=1.570796 effort=3 velocity=20 -> lower=-1.570796 upper=0.5 effort=3 velocity=20

File: urdf/arm/arm.urdf.xacro (robot description, xacro)
@@ -63,5 +63,5 @@
             <parent link="arm_${side}_1_link" />
             <child link="arm_${side}_2_link" />
-            <limit lower="${-90*deg_to_rad}" upper="${90*deg_to_rad}" effort="50" velocity="4" />
+            <limit lower="${-90*deg_to_rad}" upper="0.5" effort="50" velocity="4" />
         </joint>
         <link name="arm_${side}_3_link">

Commit message: Add target_indicator model, add color to arm end marker

File: robots/arm_standalone.urdf (robot description, URDF)
Before this commit: robot lobot, 10 links, 9 joints
Links:
- link grip_end_point: geometry visual sphere radius=0.004
